Commit message: test noflat

File: resources/robots/Pikachu_V025/urdf/Pikachu_V025.urdf (robot description, URDF)
Before this commit: robot Pikachu_V025, 19 links, 18 joints
Links:
- added link left_foot, mass 1e-9
- added link right_foot, mass 1e-9
- added link trunk, mass 1e-9
Joints:
- added joint left_foot_frame: type fixed, parent left_ankle_link, child left_foot, origin xyz=0 0 -0.05 rpy=0 0 0, axis 0 0 0
- added joint right_foot_frame: type fixed, parent right_ankle_link, child right_foot, origin xyz=0 0 -0.05 rpy=0 0 0, axis 0 0 0
- added joint trunk_frame: type fixed, parent base_link, child trunk, origin xyz=0 0 0.1 rpy=0 0 0, axis 0 0 0
